File: hardware/stm32-grbl.kicad_sch (KiCad schematic)
At the start: 104 parts, among them J1 USB_B, J10 LIMIT_X, J11 LIMIT_Y, J12 LIMIT_Z, J13 PROBE, J14 SP_DIR, J15 LIGHT, J16 RELAY_1, J17 RELAY_2, J18 RELAY_3, J19 RELAY_4, J2 FLOOD, J20 RELAY_POWER, J21 POWER, J3 SWD, J4 MIST, J5 RESET, J6 FEED_HOLD, J7 CYCLE_START, J8 SAFETY_DOOR, J9 SP_ENA, Q1 IRFR540N, Q2 IRFR540N, Q3 IRFR540N, Q4 IRFR540N, Q5 IRFR540N, SW1 RESET, U1 AMS1117-3.3, U10 PC817, U11 PC817, U2 STM32F103C8Tx, U3 PC817, U4 PC817, U5 PC817, U6 PC817, U7 PC817, U8 PC817, U9 PC817, Y1 8Mhz

Commit message: HW update
Parts:
- gave numbers to parts that had none: 3
Changed lines of the file:
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@@
   (symbol (lib_id "Connector:Conn_01x04_Male") (at 268.605 40.64 180) (unit 1)
     (in_bom yes) (on_board yes)
-    (property "Reference" "J?" (id 0) (at 269.24 38.735 0)
+    (property "Reference" "J22" (id 0) (at 269.24 38.735 0)
       (effects (font (size 1.27 1.27)) (justify right))
     )
@@
   (symbol (lib_id "Connector:Conn_01x04_Male") (at 268.605 88.9 180) (unit 1)
     (in_bom yes) (on_board yes)
-    (property "Reference" "J?" (id 0) (at 269.24 86.36 0)
+    (property "Reference" "J23" (id 0) (at 269.24 86.36 0)
       (effects (font (size 1.27 1.27)) (justify right))
     )
@@
   (symbol (lib_id "Connector:Conn_01x04_Male") (at 268.605 137.16 180) (unit 1)
     (in_bom yes) (on_board yes)
-    (property "Reference" "J?" (id 0) (at 269.24 134.62 0)
+    (property "Reference" "J24" (id 0) (at 269.24 134.62 0)
       (effects (font (size 1.27 1.27)) (justify right))
     )
@@
     )
     (path "/1d49ec3c-eadf-4c77-9805-dec4ebef2ac1"
-      (reference "J?") (unit 1) (value "X_STEPPER") (footprint "Connector_JST:JST_EH_B4B-EH-A_1x04_P2.50mm_Vertical")
+      (reference "J22") (unit 1) (value "X_STEPPER") (footprint "Connector_JST:JST_EH_B4B-EH-A_1x04_P2.50mm_Vertical")
     )
     (path "/4422ef2a-acc8-4f1b-b12e-c5a5d2593172"
-      (reference "J?") (unit 1) (value "Y_STEPPER") (footprint "Connector_JST:JST_EH_B4B-EH-A_1x04_P2.50mm_Vertical")
+      (reference "J23") (unit 1) (value "Y_STEPPER") (footprint "Connector_JST:JST_EH_B4B-EH-A_1x04_P2.50mm_Vertical")
     )
     (path "/aea05e1d-c8e5-4863-ad26-f0b961a8d385"
-      (reference "J?") (unit 1) (value "Z_STEPPER") (footprint "Connector_JST:JST_EH_B4B-EH-A_1x04_P2.50mm_Vertical")
+      (reference "J24") (unit 1) (value "Z_STEPPER") (footprint "Connector_JST:JST_EH_B4B-EH-A_1x04_P2.50mm_Vertical")
     )
     (path "/9c6beff8-c008-47d9-9802-e5b7a3a7e8cb"
